File: kicad/split-keyboard-kicad.kicad_pcb (KiCad board)
At the start: 2 copper layers, 235 x 154 mm, 109 parts, among them SW1 SW_Push, SW10 SW_Push, SW11 SW_Push, SW12 SW_Push, SW13 SW_Push, SW14 SW_Push, SW15 SW_Push, SW16 SW_Push, SW17 SW_Push, SW18 SW_Push, SW19 SW_Push, SW2 SW_Push, SW20 SW_Push, SW21 SW_Push, SW22 SW_Push, SW23 SW_Push, SW24 SW_Push, SW25 SW_Push, SW26 SW_Push, SW27 SW_Push, SW28 SW_Push, SW29 SW_Push, SW3 SW_Push, SW30 SW_Push, SW31 SW_Push, SW32 SW_Push, SW33 SW_Push, SW34 SW_Push, SW35 SW_Push, SW36 SW_Push, SW37 SW_Push, SW38 SW_Push, SW39 SW_Push, SW4 SW_Push, SW40 SW_Push, SW41 SW_Push, SW42 SW_Push, SW43 SW_Push, SW44 SW_Push, SW46 RotaryEncoder, SW47 RotaryEncoder, SW5 SW_Push, SW6 SW_Push, SW7 SW_Push, SW8 SW_Push, SW9 SW_Push, U1 DM-OLED096-636, U2 DM-OLED096-636

Commit message: updated readme
Parts:
- removed the G*** at (119.5, 66.9)
- removed the G*** at (195.5, 65.3)
- removed the G*** at (233.5, 98.6)
- removed the G*** at (232.2, 130.7)
- removed the G*** at (248.0, 40.5)
- removed the G*** at (243.9, 162.3)
- removed the G*** at (59.8, 136.0)
- removed the G*** at (124.7, 39.6)
- removed the G*** at (180.2, 115.1)
- removed the G*** at (68.5, 67.0)
- removed the G*** at (183.1, 39.9)
- removed the G*** at (65.6, 161.7)
- removed the G*** at (68.4, 41.3)
- removed the G*** at (117.0, 126.0)
- removed the G*** at (184.2, 149.6)
- added G***: LOGO, kicad-image:batman-og, B.Cu at (234.3, 32.7)
- added G***: LOGO, kicad-image:batman-og, B.Cu at (234.4, 181.8)
- added G***: LOGO, LOGO, B.Cu at (67.8, 96.0)
- added G***: LOGO, kicad-image:batman-og, B.Cu at (110.8, 37.4)
- added G***: LOGO, kicad-image:batman-og, B.Cu at (174.9, 181.4)
- added G***: LOGO, kicad-image:batman-og, B.Cu at (149.5, 31.8)
- added G***: LOGO, LOGO, B.Cu at (189.9, 90.9)
- added G***: LOGO, kicad-image:batman-og, B.Cu at (108.6, 161.1)
- added G***: LOGO, kicad-image:batman-og, B.Cu at (35.7, 179.1)
- added G***: LOGO, kicad-image:batman-og, B.Cu at (36.0, 34.5)
- moved SW47 112.1 mm to (24.0, 37.5)
- moved SW23 101.2 mm to (93.0, 168.9)
- moved SW46 89.0 mm to (224.4, 36.2)
- moved SW33 84.9 mm to (54.1, 111.9)
- moved SW27 84.7 mm to (34.9, 111.9)
- moved SW34 84.7 mm to (54.3, 131.4)
- moved SW28 84.5 mm to (35.0, 131.4)
- moved D14 67.8 mm to (194.7, 183.0)
- moved D6 67.8 mm to (183.9, 183.0)
- moved D16 63.4 mm to (195.0, 177.0)
- moved D8 63.2 mm to (184.4, 177.0)
- moved D15 62.3 mm to (195.5, 170.5)
- moved D7 62.3 mm to (184.7, 170.5)
- moved SW19 61.1 mm to (233.6, 131.5)
- moved U1 59.7 mm to (181.5, 48.5)
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Routing:
- net /left/col1: track 173.0 -> 372.3 mm
- net /left/row2: track 228.9 -> 407.3 mm, vias 1 -> 0
- net /right/col1: track 33.0 -> 192.2 mm
- net Net-(D30-A): track 147.9 -> 282.1 mm, vias 2 -> 0
- net Net-(D14-A): track 0.00 -> 130.3 mm
- net /right/row3: track 49.7 -> 177.4 mm, vias 0 -> 1
- net /right/row2: track 38.5 -> 160.1 mm, vias 0 -> 1
- net /left/row4: track 301.7 -> 420.8 mm
- net /left/leftPower: track 202.2 -> 95.0 mm
- net /left/col5: track 242.9 -> 136.0 mm, vias 1 -> 0
- net /left/sda: track 188.1 -> 82.3 mm, vias 1 -> 0
- net /left/row1: track 237.1 -> 342.4 mm
- net Net-(D28-A): track 38.7 -> 143.6 mm, vias 0 -> 1
- net Net-(D7-A): track 0.00 -> 102.1 mm
- net Net-(D15-A): track 0.00 -> 97.1 mm
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Other:
- board size 235 x 154 mm -> 230.5 x 167.5 mm
- board text added: "-by AYUSH"
- board text removed: "-by Ayush"
